File: ttgo-baseplate/ttgo-baseplate/ttgo-baseplate.sch (KiCad schematic (older format))
At the start: 4 parts, among them J1 Conn_02x16_Odd_Even, J2 Conn_02x16_Odd_Even, J3 Conn_02x10_Odd_Even, J4 Conn_01x05

Commit message: - Adjusted T4 size and drilling holes on footprint - Changed footprint of the TTGO T4 expansion connector to match pn numbering of schematic. - Signals on the TTGO T4 were mirrorred top bottom, corrected order. - TTGO-T4 to Wemos mapping was not followed making most Dx signals on the inner Wemos connector unusable. - Added jumpers to replace I2C by other signals. Cut them if you want to use the I2C connector on the board. - Added ground planes at both sides. Board is now 2 layers. - Used proper drill holes. The mounting holes did not appear in a drilling file. Not a clue if they can be done as an edge cut. But this will certainly work.\ - Lots of small changes hre and there.
Parts:
- added JP1: SDA, Jumper:SolderJumper-2_P1.3mm_Bridged_RoundedPad1.0x1.5mm, symbol Jumper:SolderJumper_2_Bridged
- added JP2: SCL, Jumper:SolderJumper-2_P1.3mm_Bridged_RoundedPad1.0x1.5mm, symbol Jumper:SolderJumper_2_Bridged
- added MH1, MH2, MH3, MH4: MountingHole, MountingHole:MountingHole_3.2mm_M3, symbol Mechanical:MountingHole
- J3: symbol Connector_Generic:Conn_02x10_Odd_Even -> Connector_Generic:Conn_02x10_Counter_Clockwise
Connections:
- no-connect marks 2 -> 3
Changed lines of the file:
@@
 EESchema Schematic File Version 4
-EELAYER 30 0
+LIBS:ttgo-baseplate-cache
+EELAYER 26 0
 EELAYER END
 $Descr A4 11693 8268
 encoding utf-8
 Sheet 1 1
-Title ""
-Date ""
-Rev ""
-Comp ""
-Comment1 ""
-Comment2 ""
+Title "TTGO-T4-Base Plate"
+Date "2020-02-10"
+Rev "1.1"
+Comp "Sensemakers Amsterdam"
+Comment1 "Revisions: Gijs Mos"
+Comment2 "Author: Karijn Wessing"
 Comment3 ""
 Comment4 ""
@@
 $EndComp
 $Comp
-L Connector_Generic:Conn_02x10_Odd_Even J3
+L Connector_Generic:Conn_02x10_Counter_Clockwise J3
 U 1 1 5E3BEFF0
 P 6725 1500
@@
 	1    0    0    -1
 $EndComp
-Text Label 7225 2725 2    50   ~ 0
-3.3V
 Text Label 7225 3025 2    50   ~ 0
 5V
@@
 Text Label 7225 2925 2    50   ~ 0
 SDA
+Text Label 6525 2000 2    50   ~ 0
+5V
+Text Label 6525 1900 2    50   ~ 0
+GND
+Text Label 7025 1900 0    50   ~ 0
+3.3V
+Text Label 6525 1700 2    50   ~ 0
+IO19
+Text Label 6525 1600 2    50   ~ 0
+RXD
+Text Label 6525 1500 2    50   ~ 0
+TXD
+Text Label 6525 1400 2    50   ~ 0
+IO17
+Text Label 6525 1300 2    50   ~ 0
+IO32
+Text Label 6525 1200 2    50   ~ 0
+IO34
 Text Label 6525 1100 2    50   ~ 0
-5V
-Text Label 6525 1200 2    50   ~ 0
-GND
-Text Label 6525 1300 2    50   ~ 0
-3.3V
-Text Label 6525 1400 2    50   ~ 0
-IO19
-Text Label 6525 1500 2    50   ~ 0
-RXD
-Text Label 6525 1600 2    50   ~ 0
-TXD
-Text Label 6525 1700 2    50   ~ 0
-IO25
-Text Label 6525 1800 2    50   ~ 0
+SVN
+Text Label 7025 1100 0    50   ~ 0
+SVP
+Text Label 7025 1200 0    50   ~ 0
+RST
+Text Label 7025 1300 0    50   ~ 0
+IO05
+Text Label 7025 1400 0    50   ~ 0
+IO18
+Text Label 7025 1500 0    50   ~ 0
+GND
+Text Label 7025 1600 0    50   ~ 0
+IO26
+Text Label 7025 1700 0    50   ~ 0
+GND
+Text Label 7025 1800 0    50   ~ 0
+IO23
+NoConn ~ 7025 2000
+NoConn ~ 7225 2725
+$Comp
+L Mechanical:MountingHole MH1
+U 1 1 5E40BFB7
+P 7300 3550
+F 0 "MH1" H 7400 3596 50  0000 L CNN
+F 1 "MountingHole" H 7400 3505 50  0000 L CNN
+F 2 "MountingHole:MountingHole_3.2mm_M3" H 7300 3550 50  0001 C CNN
+F 3 "~" H 7300 3550 50  0001 C CNN
+	1    7300 3550
+	1    0    0    -1
+$EndComp
+$Comp
+L Mechanical:MountingHole MH3
+U 1 1 5E40C0AD
+P 8050 3550
+F 0 "MH3" H 8150 3596 50  0000 L CNN
+F 1 "MountingHole" H 8150 3505 50  0000 L CNN
+F 2 "MountingHole:MountingHole_3.2mm_M3" H 8050 3550 50  0001 C CNN
+F 3 "~" H 8050 3550 50  0001 C CNN
+	1    8050 3550
+	1    0    0    -1
+$EndComp
+$Comp
+L Mechanical:MountingHole MH2
+U 1 1 5E40C0EF
+P 7300 3825
+F 0 "MH2" H 7400 3871 50  0000 L CNN
+F 1 "MountingHole" H 7400 3780 50  0000 L CNN
+F 2 "MountingHole:MountingHole_3.2mm_M3" H 7300 3825 50  0001 C CNN
+F 3 "~" H 7300 3825 50  0001 C CNN
+	1    7300 3825
+	1    0    0    -1
+$EndComp
+$Comp
+L Mechanical:MountingHole MH4
+U 1 1 5E40C125
+P 8050 3825
+F 0 "MH4" H 8150 3871 50  0000 L CNN
+F 1 "MountingHole" H 8150 3780 50  0000 L CNN
+F 2 "MountingHole:MountingHole_3.2mm_M3" H 8050 3825 50  0001 C CNN
+F 3 "~" H 8050 3825 50  0001 C CNN
+	1    8050 3825
+	1    0    0    -1
+$EndComp
+NoConn ~ 6525 1800
+$Comp
+L Jumper:SolderJumper_2_Bridged JP1
+U 1 1 5E4167ED
+P 5775 1200
+F 0 "JP1" H 5775 1405 50  0000 C CNN
+F 1 "SDA" H 5775 1314 50  0000 C CNN
+F 2 "Jumper:SolderJumper-2_P1.3mm_Bridged_RoundedPad1.0x1.5mm" H 5775 1200 50  0001 C CNN
+F 3 "~" H 5775 1200 50  0001 C CNN
+	1    5775 1200
+	1    0    0    -1
+$EndComp
+$Comp
+L Jumper:SolderJumper_2_Bridged JP2
+U 1 1 5E416887
+P 5775 1575
+F 0 "JP2" H 5775 1780 50  0000 C CNN
+F 1 "SCL" H 5775 1689 50  0000 C CNN
+F 2 "Jumper:SolderJumper-2_P1.3mm_Bridged_RoundedPad1.0x1.5mm" H 5775 1575 50  0001 C CNN
+F 3 "~" H 5775 1575 50  0001 C CNN
+	1    5775 1575
+	1    0    0    -1
+$EndComp
+Text Label 5925 1200 0    50   ~ 0
 IO32
-Text Label 6525 1900 2    50   ~ 0
+Text Label 5925 1575 0    50   ~ 0
 IO34
-Text Label 6525 2000 2    50   ~ 0
-SVN
-Text Label 7025 2000 0    50   ~ 0
-SVP
-Text Label 7025 1900 0    50   ~ 0
-RST
-Text Label 7025 1800 0    50   ~ 0
-IO35
-Text Label 7025 1700 0    50   ~ 0
-IO33
-Text Label 7025 1600 0    50   ~ 0
-GND
-Text Label 7025 1500 0    50   ~ 0
-IO00
-Text Label 7025 1400 0    50   ~ 0
-GND
-Text Label 7025 1300 0    50   ~ 0
-IO04
-NoConn ~ 7025 1200
-NoConn ~ 7025 1100
+Text Label 5625 1200 2    50   ~ 0
+SDA
+Text Label 5625 1575 2    50   ~ 0
+SCL
 $EndSCHEMATC
